File: ezPLA.sch (KiCad schematic (older format))
At the start: 4 parts, among them J1 JTAG-10, J2 Power, J3 PLA-headers, U2 EPM7032

Commit message: Update KiCad files
Parts:
- J1: footprint C64_PLA:IDC-Header_2x05_P2.54mm_Custom -> ezPLA footprints:IDC-Header_2x05_P2.54mm_Custom
- J3: footprint C64_PLA:DIP-28_W15.24mm_mirrored -> ezPLA footprints:DIP-28_W15.24mm_mirrored; symbol C64:PLA-headers -> C64_ezPLA:PLA-headers
Changed lines of the file:
@@
 F 0 "J1" H 7350 4050 50  0000 R CNN
 F 1 "JTAG-10" H 7800 3400 50  0000 R CNN
-F 2 "C64_PLA:IDC-Header_2x05_P2.54mm_Custom" V 7550 3600 50  0001 C CNN
+F 2 "ezPLA footprints:IDC-Header_2x05_P2.54mm_Custom" V 7550 3600 50  0001 C CNN
 F 3 " ~" H 6425 2900 50  0001 C CNN
 	1    7700 3450
@@
 Connection ~ 7650 4750
 $Comp
-L C64:PLA-headers J3
+L C64_ezPLA:PLA-headers J3
 U 1 1 6115D0F0
 P 3050 3850
 F 0 "J3" H 2950 4650 50  0000 L CNN
 F 1 "PLA-headers" H 3100 4800 50  0000 L CNN
-F 2 "C64_PLA:DIP-28_W15.24mm_mirrored" H 3050 3950 50  0001 C CNN
+F 2 "ezPLA footprints:DIP-28_W15.24mm_mirrored" H 3050 3950 50  0001 C CNN
 F 3 "~" H 3050 3950 50  0001 C CNN
 	1    3050 3850
@@
 	3050 4500 2950 4500
 $Comp
-L C64:PLA-headers J3
+L C64_ezPLA:PLA-headers J3
 U 2 1 6117326B
 P 3800 3850
 F 0 "J3" H 3650 4650 50  0000 L CNN
 F 1 "PLA-headers" H 3892 3066 50  0001 C CNN
-F 2 "C64_PLA:DIP-28_W15.24mm_mirrored" H 3800 3950 50  0001 C CNN
+F 2 "ezPLA footprints:DIP-28_W15.24mm_mirrored" H 3800 3950 50  0001 C CNN
 F 3 "~" H 3800 3950 50  0001 C CNN
 	2    3800 3850
